File: board/plzoreg.kicad_sch (KiCad schematic)
At the start: 53 parts, among them J1 IN, J2 OUT, J3 Heatsink Earth, Q1 BTA24-600C, U1 HLK-PM03, U2 H11AA1, U3 MOC3023M, U4 PY32F030K1xTx, X1 SWD

Commit message: WIP
Parts:
- added C14: 100n, Capacitor_SMD:C_0805_2012Metric_Pad1.18x1.45mm_HandSolder, symbol Device:C
- added H1, H2, H3, H4: MountingHole, MountingHole:MountingHole_4.3mm_M4_Pad_Via, symbol Mechanical:MountingHole
- added R19: 47k 1%, Resistor_SMD:R_0805_2012Metric_Pad1.20x1.40mm_HandSolder, symbol Device:R
- added R20: 1k5, Resistor_SMD:R_0805_2012Metric_Pad1.20x1.40mm_HandSolder, symbol Device:R
- added TH1: 3950, Connector_PinHeader_2.54mm:PinHeader_1x02_P2.54mm_Vertical, symbol Device:Thermistor_NTC
- added TP6: TSENSE, TestPoint:TestPoint_THTPad_D2.0mm_Drill1.0mm, symbol Connector:TestPoint
- J3: footprint Connector_Pin:Pin_D1.0mm_L10.0mm -> Connector_Wire:SolderWire-1.5sqmm_1x01_D1.7mm_OD3.9mm
- R7: footprint Resistor_SMD:R_0805_2012Metric_Pad1.20x1.40mm_HandSolder -> Resistor_THT:R_Axial_DIN0207_L6.3mm_D2.5mm_P10.16mm_Horizontal
- TP5: value ADC -> VSENSE
Connections:
- net DISP_CC1: now also U4.5 (PF3); no longer U4.26 (PB3)
- net DISP_CC2: now also U4.28 (PB5); no longer U4.27 (PB4)
- net DISP_CC3: now also U4.27 (PB4); no longer U4.28 (PB5)
- net GND: now also C14.1, TH1.2
- net MAINS_L_IN: now also J1.1 (Pin_1); no longer J1.3 (Pin_3)
- net VCC: now also R19.1
- net ZCD: now also U4.20 (PA10-OSC32IN); no longer U4.15 (PB1)
- net at C4.1, C6.1, D1.1 (K)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: no longer TP5.1
- net ADC renamed VSENSE
- net VSENSE: now also TP5.1
- net MAIN_PEN renamed MAIN_PE
- net MAIN_PE: now also J1.3 (Pin_3); no longer J1.1 (Pin_1)
- new net: R19.2, R20.1, TH1.1
- new net TSENSE: C14.2, R20.2, TP6.1, U4.15 (PB1)
- no-connect marks 10 -> 9
Other:
- moved on the sheet: BTN1, BTN2, C11, C12, C4, C6, D1, D2A, D2B, J3, R10, R2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

Commit message: WIP
Parts:
- J3: value Heatsink Earth -> Heatsink PE
Changed lines of the file:
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@@
 			)
 		)
-		(property "Value" "Heatsink Earth"
+		(property "Value" "Heatsink PE"
 			(at 52.07 189.2299 0)
 			(effects

Commit message: WIP
Parts:
- removed C4: 10u, Capacitor_SMD:C_0805_2012Metric_Pad1.18x1.45mm_HandSolder, symbol Device:C
- removed D1: DSK14, Diode_SMD:D_SOD-123, symbol Device:D
- removed D2: BAT54S, Package_TO_SOT_SMD:SOT-23, symbol Device:D_Dual_Series_AKC_Split
- removed R4: 10k/0.5W, Resistor_THT:R_Axial_DIN0411_L9.9mm_D3.6mm_P12.70mm_Horizontal, symbol Device:R
- added R9: 10k, Resistor_SMD:R_0805_2012Metric_Pad1.20x1.40mm_HandSolder, symbol Device:R
- added U3: LTV-817S, Package_DIP:SMDIP-4_W9.53mm, symbol Isolator:LTV-817S
- C4: renamed from C6; value 100n -> 1u
- R4: renamed from R2; value 510k/0.5W -> 330k/0.5W
- R5: renamed from R3; value 510k/0.5W -> 330k/0.5W
- renumbered C14 to C10, C7 to C6, C8 to C7, C9 to C8, C10 to C9, J3 to J2, J2 to J3, R19 to R11, R20 to R12, R11 to R13, R12 to R14, R13 to R15, R14 to R16, R15 to R17, R16 to R18, R17 to R19, R5 to R2, R18 to R20, R6 to R3, R7 to R6, R8 to R7, R9 to R8, U3 to U4, U4 to U5
Connections:
- net GND: now also U3.3; no longer R5.2
- net MAINS_L_IN: now also R5.1; no longer R4.1
- net MAINS_N: now also R4.1; no longer R5.1
- net VCC: now also R9.1
- net at R4.2: now also U3.1
- net at C4.1, R10.1: now also R9.2, U3.4
- new net: R5.2, U3.2
Other:
- moved on the sheet: C4, R10, R4, R5, TP5

Commit message: WIP
Parts:
- removed C13: 100n, Capacitor_SMD:C_0805_2012Metric_Pad1.18x1.45mm_HandSolder, symbol Device:C
- U5: value PY32F030K1xTx -> PY32F030K2xTx; symbol MCU_Puya_PY32F:PY32F030K1xTx -> MCU_Puya_PY32F:PY32F030K2xTx
Connections:
- net DISP_CC1: now also U5.25 (PA15); no longer U5.5 (PF3)
- net DISP_CC2: now also U5.26 (PB3); no longer U5.28 (PB5)
- net GND: no longer U5.32 (VSS)
- net VCC: no longer U5.17 (VCC)
- net at U5.10 (PA4): now also R18.1; no longer R17.1
- net at U5.11 (PA5): now also R19.1; no longer R18.1
- net at U5.12 (PA6): now also R20.1; no longer R19.1
- net at U5.13 (PA7): no longer R20.1
- net at R13.1: now also U5.32 (PB8); no longer U5.6 (PA0)
- net at R14.1: now also U5.6 (PA0); no longer U5.7 (PA1)
- net at R15.1: now also U5.7 (PA1); no longer U5.8 (PA2)
- net at R16.1: now also U5.8 (PA2); no longer U5.9 (PA3)
- new net: R17.1, U5.9 (PA3)
- no-connect marks 9 -> 11
Other:
- moved on the sheet: R13, R14, R15, R16, R17, R18, R19, R20

Commit message: WIP
Parts:
- removed U2: H11AA1, Package_DIP:DIP-6_W8.89mm_SMDSocket_LongPads, symbol Isolator:H11AA1
- added U6: LTV-354T, Package_SO:SO-4_4.4x3.6mm_P2.54mm, symbol Isolator:LTV-354T
- C4: value 1u -> 10u
- R9: value 10k -> 1k5
Connections:
- net GND: now also U6.3
- net ZCD: now also U6.4
- net at R2.2: now also U6.1
- net at R3.1: now also U6.2
- no-connect marks 11 -> 10
Other:
- moved on the sheet: C2, R8, TP2

Commit message: WIP
Parts:
- added H5, H6: MountingHole, MountingHole:MountingHole_3.7mm, symbol Mechanical:MountingHole
Changed lines of the file:
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@@
+	)
+	(symbol
+		(lib_id "Mechanical:MountingHole")
+		(at 152.4 185.42 0)
+		(unit 1)
+		(exclude_from_sim no)
+		(in_bom no)
+		(on_board yes)
+		(dnp no)
+		(property "Reference" "H5"
+			(at 155.448 185.42 0)
+			(effects
+				(font
+					(size 1.27 1.27)
+				)
+				(justify left)
+			)
+		)
+		(property "Value" "MountingHole"
+			(at 154.94 186.6899 0)
+			(effects
+				(font
+					(size 1.27 1.27)
+				)
+				(justify left)
+				(hide yes)
+			)
+		)
+		(property "Footprint" "MountingHole:MountingHole_3.7mm"
+			(at 152.4 185.42 0)
+			(effects
+				(font
+					(size 1.27 1.27)
+				)
+				(hide yes)
+			)
+		)
+		(property "Datasheet" "~"
+			(at 152.4 185.42 0)
+			(effects
+				(font
+					(size 1.27 1.27)
+				)
+				(hide yes)
+			)
+		)
+		(property "Description" "Mounting Hole without connection"
+			(at 152.4 185.42 0)
+			(effects
+				(font
+					(size 1.27 1.27)
+				)
+				(hide yes)
+			)
+		)
+		(instances
+			(project "plzoreg"
+				(path "/ec1239b0-05b9-4998-8e2e-5748175a8483"
+					(reference "H5")
+					(unit 1)
+				)
+			)
+		)
 	)
 	(symbol
@@
 					(unit 1)
 				)
+			)
+		)
+	)
+	(symbol
+		(lib_id "Mechanical:MountingHole")
+		(at 152.4 190.5 0)
+		(unit 1)
+		(exclude_from_sim no)
+		(in_bom no)
+		(on_board yes)
+		(dnp no)
+		(property "Reference" "H6"
+			(at 155.448 190.5 0)
+			(effects
+				(font
+					(size 1.27 1.27)
+				)
+				(justify left)
+			)
+		)
+		(property "Value" "MountingHole"
+			(at 154.94 191.7699 0)
+			(effects
+				(font
+					(size 1.27 1.27)
+				)
+				(justify left)
+				(hide yes)
+			)
+		)
+		(property "Footprint" "MountingHole:MountingHole_3.7mm"
+			(at 152.4 190.5 0)
+			(effects
+				(font
+					(size 1.27 1.27)
+				)
+				(hide yes)
+			)
+		)
+		(property "Datasheet" "~"
+			(at 152.4 190.5 0)
+			(effects
+				(font
+					(size 1.27 1.27)
+				)
+				(hide yes)
+			)
+		)
+		(property "Description" "Mounting Hole without connection"
+			(at 152.4 190.5 0)
+			(effects
+				(font
+					(size 1.27 1.27)
+				)
+				(hide yes)
+			)
+		)
+		(instances
+			(project "plzoreg"
+				(path "/ec1239b0-05b9-4998-8e2e-5748175a8483"
+					(reference "H6")
+					(unit 1)
+				)

Commit message: WIP
Parts:
- added J4: AUX, Connector_IDC:IDC-Header_2x07_P2.54mm_Vertical, symbol Connector_Generic:Conn_02x07_Odd_Even
Connections:
- net GND: now also J4.13 (Pin_13), J4.14 (Pin_14)
- net VCC: now also J4.1 (Pin_1), J4.2 (Pin_2)
- net AUX_PA7: now reaches U5.13 (PA7)
- net AUX_PA7: now also J4.11 (Pin_11)
- net AUX_PB2: now reaches U5.17 (PB2)
- net AUX_PB2: now also J4.3 (Pin_3)
- net AUX_PA9: now reaches U5.19 (PA9-OSC32OUT)
- net AUX_PA9: now also J4.5 (Pin_5)
- net AUX_PF0: now reaches U5.2 (PF0-OSCIN)
- net AUX_PF0: now also J4.4 (Pin_4)
- net AUX_PB5: now reaches U5.28 (PB5)
- net AUX_PB5: now also J4.12 (Pin_12)
- net AUX_PB6: now reaches U5.29 (PB6)
- net AUX_PB6: now also J4.10 (Pin_10)
- net AUX_PF1: now reaches U5.3 (PF1-OSCOUT)
- net AUX_PF1: now also J4.7 (Pin_7)
- net AUX_PB7: now reaches U5.30 (PB7)
- net AUX_PB7: now also J4.8 (Pin_8)
- net AUX_PF4: now reaches U5.31 (PF4-BT0)
- net AUX_PF4: now also J4.6 (Pin_6)
- net AUX_PF3: now reaches U5.5 (PF3)
- net AUX_PF3: now also J4.9 (Pin_9)
- no-connect marks 10 -> 0
Other:
- moved on the sheet: R13

Commit message: WIP
Parts:
- R9: value 1k5 -> 10k
Changed lines of the file:
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@@
 			)
 		)
-		(property "Value" "1k5"
+		(property "Value" "10k"
 			(at 109.22 114.3 90)
 			(effects
